File: om27_strumplate/kicad/om27_strumplate/om27_strumplate.kicad_pcb (KiCad board)
At the start: 2 copper layers, 112.1 x 159.1 mm, 0 parts

Commit message: Fixes after JLC feedback
Other:
- board text added: "Add stiffener at filled white areas Material: Polyimide Total thickness Golden Finger: 0.32mm Gold Finger on top-side"
- board text added: "Bottom Side"
- board text added: "Top Side"
- board text removed: "Add stiffener at filled white areas Material: Polyimide Total thickness: 0.3mm Gold teeth on front-side"
Changed lines of the file:
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@@
 	(gr_poly
 		(pts
-			(xy 110.33 164.04) (xy 88.316877 164.04) (xy 88.316877 19.56179) (xy 110.33 19.56179)
+			(xy 109.49 164.04) (xy 88.986877 164.04) (xy 88.986877 19.56179) (xy 109.49 19.56179)
 		)
 		(stroke
@@
 	(gr_poly
 		(pts
-			(xy 140.696149 54.970878) (xy 125.956861 54.970878) (xy 125.956861 39.326224) (xy 140.696149 39.326224)
+			(xy 141.596149 54.970878) (xy 125.956861 54.970878) (xy 125.956861 39.656224) (xy 141.596149 39.656224)
 		)
 		(stroke
 			(width 0.909496)
 			(type solid)
+		)
+		(fill yes)
+		(layer "F.Mask")
+	)
+	(gr_rect
+		(start 191.9 69.63)
+		(end 194.085278 88.47)
+		(stroke
+			(width 0.2)
+			(type default)
 		)
 		(fill yes)
@@
 			(xy 83.013733 171.344611) (xy 82.929901 171.227156) (xy 82.850806 171.10278) (xy 82.776537 170.971566)
 			(xy 82.707185 170.833597) (xy 82.642838 170.688957) (xy 82.522886 168.814863) (xy 82.476672 164.074394)
-			(xy 87.576858 164.074394) (xy 109.589979 164.074394) (xy 109.589979 55.354976) (xy 125.328533 55.354976)
-			(xy 140.804607 55.354976) (xy 140.804607 39.01074) (xy 125.328564 39.01074) (xy 125.328533 55.354976)
-			(xy 109.589979 55.354976) (xy 109.589979 19.595886) (xy 87.576858 19.595886) (xy 87.576858 164.074394)
+			(xy 87.576858 164.074394) (xy 109.959979 164.074394) (xy 109.959979 55.354976) (xy 125.328533 55.354976)
+			(xy 142.254607 55.354976) (xy 142.254607 39.01074) (xy 125.328564 39.01074) (xy 125.328533 55.354976)
+			(xy 110.049979 55.354976) (xy 110.049979 19.595886) (xy 88.606858 19.595886) (xy 88.606858 164.074394)
 			(xy 82.476672 164.074394) (xy 82.451241 161.465812) (xy 82.383926 115.678886) (xy 82.281601 60.560847)
 			(xy 82.212387 32.87518) (xy 82.214401 14.798767) (xy 82.396805 14.414794) (xy 82.440994 14.327837)
@@
 		(layer "User.1")
 	)
-	(gr_text "Add stiffener at filled white areas\nMaterial: Polyimide\nTotal thickness: 0.3mm\nGold teeth on front-side"
+	(gr_text "Add stiffener at filled white areas\nMaterial: Polyimide\nTotal thickness Golden Finger: 0.32mm\nGold Finger on top-side"
 		(at 152.58 106.59 0)
 		(layer "User.1")
@@
 		)
 	)
+	(gr_text "Bottom Side"
+		(at 181.32 91.63 0)
+		(layer "User.1")
+		(effects
+			(font
+				(size 1.5 1.5)
+				(thickness 0.3)
+				(bold yes)
+			)
+			(justify left bottom)
+		)
+	)
+	(gr_text "Top Side"
+		(at 145.78 102.95 90)
+		(layer "User.1")
+		(effects
+			(font
+				(size 1.5 1.5)
+				(thickness 0.3)
+				(bold yes)
+			)
+			(justify left bottom)
+		)
+	)
 	(group ""
 		(members "16fde469-888c-4869-9b1b-6ce320c43efb" "1ec7ea7e-14ec-4762-8a8e-9f16705325da"
@@
 	)
 	(group ""
-		(members "324bfde8-907c-42b0-baa9-2f00f5fd3c8e" "c31de017-9de9-4bfa-b396-82a21ed98ee4")
-	)
-	(group ""
 		(members "a74320f2-3234-4452-97f2-a9609de735e6" "c8d32107-89f9-4ee9-a582-6f4fc5751404"
 			"cae2a0fb-48a3-4608-b20e-472bf5f8c177"
 		)
 	)
-	(group ""
-		(members "650c7b21-2890-4111-9791-f8e4ff9e2f82" "9d44d77f-64f5-436b-90e6-d15928405e2c"
-			"c7554a0a-db39-4d9c-b7f8-0db8c098ff15" "dc27789c-1f6c-44e1-bdf4-c3a4eb16dcc4"
-		)
-	)
